File: tamago.kicad_pcb (KiCad board)
At the start: 2 copper layers, 75.8 x 71.9 mm, 16 parts, among them J1 USB_C_Receptacle_USB2.0_16P, J2 OLED, J3 Rotary Encoder, J4 INMP441, SW1 SW_Push, SW2 SW_Push, U1 AP2112K-3.3, U2 ESP32-C3-MINI-1, U3 DHT11

Commit message: pcb art
Parts:
- added G***: LOGO, pcbart-footprints:hclogo, F.Cu at (132.0, 119.5)

Commit message: new pcb art
Parts:
- added G***: LOGO, pcbart-footprints:hllogo, F.Cu at (132.0, 125.0)
- moved G*** 1.80 mm to (131.0, 118.0)
